File: hardware/FluOpti_V3.0/FluOpti_V3.0.kicad_sch (KiCad schematic)
At the start: 32 parts, among them J1 Sensor1, J2 Sensor2, J3 Conn_01x03_Pin, J4 Conn_01x02_Pin, U1 ADS1115IDGS

Commit message: esquematico
Parts:
- added C10, C11, C14, C15, C16, C17, C8, C9: 1u, symbol Device:C
- added C12, C13: C_Polarized, symbol Device:C_Polarized
- added C16, C17, C18, C19: 100n, Capacitor_SMD:C_0603_1608Metric, symbol IoWLabs:C
- added C20: 10u, Capacitor_SMD:C_0805_2012Metric, symbol IoWLabs:C
- added D111: LED, LED_SMD:LED_0603_1608Metric, symbol Device:LED
- added D3, D5, D6, D7: LED, symbol Device:LED
- added D4: D_Schottky, symbol Device:D_Schottky
- added F1: FUSE, Fuse:Fuse_1206_3216Metric, symbol IoWLabs:FUSE
- added F2: Fuse, symbol Device:Fuse
- added J10: USB_B_Micro, Connector_USB:USB_Micro-B_Amphenol_10118194_Horizontal, symbol Connector:USB_B_Micro
- added J10: LED_1, symbol Connector:Conn_01x02_Pin
- added J11: LED_2, symbol Connector:Conn_01x02_Pin
- added J12: LED_3, symbol Connector:Conn_01x02_Pin
- added J13: LED_4, symbol Connector:Conn_01x02_Pin
- added J14: H1, symbol Connector:Conn_01x02_Pin
- added J15: H2, symbol Connector:Conn_01x02_Pin
- added J5: TP-5V, symbol Connector:Conn_01x02_Pin
- added J6: TP-3.3V, symbol Connector:Conn_01x02_Pin
- added J7: TP-PWR_IN, symbol Connector:Conn_01x02_Pin
- added J8: Selector voltaje, symbol Connector_Generic:Conn_02x03_Counter_Clockwise
- added J9: TP-VCC_H1, symbol Connector:Conn_01x02_Pin
- added JP4: Jumper_2_Open, symbol Jumper:Jumper_2_Open
- added L2: 33u, symbol Device:L
- added Q1, Q2, Q3, Q4, Q5, Q6: NPN, symbol Simulation_SPICE:NPN
- added Q4: Q_Dual_NPN_NPN_BRT_E1B1C2E2B2C1, Package_TO_SOT_SMD:SOT-363_SC-70-6_Handsoldering, symbol Device:Q_Dual_NPN_NPN_BRT_E1B1C2E2B2C1
- added R13, R29, R30: 10, symbol Device:R
- added R14, R28: 1k, symbol Device:R
- added R15: 11.8k, symbol Device:R
- added R16: 15k, symbol Device:R
- added R17: 18.2k, symbol Device:R
- added R18, R19, R20, R21, R22, R23: 3.3, symbol Device:R
- added R19, R22, R23, R24: 10K, Resistor_SMD:R_0603_1608Metric, symbol IoWLabs:RES
- added R20, R21: 200, Resistor_SMD:R_0603_1608Metric, symbol IoWLabs:RES
- added R24, R25, R26: 10k, symbol Device:R
- added R25: 330, Resistor_SMD:R_0603_1608Metric, symbol IoWLabs:RES
- added R27: 2k, symbol Device:R
- added SW2, SW3: SW_DIP_x02, IoWLabs:SMD_SWITCH, symbol Switch:SW_DIP_x02
- added U10: ESP32-WROOM-32D, RF_Module:ESP32-WROOM-32, symbol RF_Module:ESP32-WROOM-32D
- added U10, U5, U6, U7, U8, U9: ${SIM.PARAMS}, symbol Simulation_SPICE:OPAMP
- added U11, U13, U3: AP2112K-3.3TRG1, IoWLabs:SOT-25, symbol IoWLabs:AP2112K-3.3TRG1-SOT25
- added U12: AD5659R, Package_SO:TSSOP-16_4.4x5mm_P0.65mm, symbol IoWLabs:AD5669R
- added U4: XL6008, Package_TO_SOT_SMD:TO-252-5_TabPin6, symbol IoWLabs:XL6008
- added U9: CH340C, Package_SO:SOIC-16_3.9x9.9mm_P1.27mm, symbol Interface_USB:CH340C
- C5: value C -> 100n
- J3: value Conn_01x03_Pin -> I2C_IN
- J4: value Conn_01x02_Pin -> PWR_IN
Connections:
- net 3.3V: now also C9.1, J6.2 (Pin_2), R13.2, R24.2, R25.2, R27.2, U12.3 (Vdd), U12.8 (V_REF), U3.5 (Vout), U4.2 (EN); no longer J1.3 (Pin_3), J2.3 (Pin_3), R10.2, R11.2
- net 5V: now also C14.1, C16.1, C8.1, J5.2 (Pin_2), U11.1 (Vin), U11.3 (EN), U13.1 (Vin), U13.3 (EN), U3.1 (Vin), U3.3 (EN)
- net GND: now also C10.2, C11.2, C12.2, C13.2, C14.2, C15.2, C16.2, C16.2, C17.2, C17.2, C18.2, C19.2, C20.2, C8.2, C9.2, D111.1 (K), D3.1 (K), D5.1 (K), D6.1 (K), D7.1 (K), J10.1 (Pin_1), J10.5 (GND), J10.6 (Shield), J11.1 (Pin_1), J12.1 (Pin_1), J13.1 (Pin_1), J14.1 (Pin_1), J15.1 (Pin_1), J5.1 (Pin_1), J6.1 (Pin_1), J7.1 (Pin_1), J9.1 (Pin_1), R14.1, R18.1, R19.1, R20.1, R21.1, R22.1, R23.1, R26.1, SW2.1, SW2.2, SW3.1, SW3.2, U10.1 (GND), U10.15 (GND), U10.38 (GND), U10.39 (GND), U10.5 (V-), U11.2 (GND), U12.14 (GND), U13.2 (GND), U3.2 (GND), U4.1 (GND), U5.5 (V-), U6.5 (V-), U7.5 (V-), U8.5 (V-), U9.1 (GND), U9.5 (V-)
- net SCL: now also R24.1, U12.16 (SCL)
- net SDA: now also R25.1, U12.15 (SDA)
- net V_PWR: now also C13.1, F2.2, J7.2 (Pin_2), R28.2, U10.4 (V+), U5.4 (V+), U6.4 (V+), U7.4 (V+), U8.4 (V+), U9.4 (V+)
- new net: Q4.2 (B1), R19.2
- new net: Q5.3 (E), R22.2, U9.2 (-)
- new net: Q5.2 (B), U9.3
- new net: JP4.1 (A), R27.1, U12.2 (A0)
- new net: Q4.3 (E), R21.2, U8.2 (-)
- new net: D6.2 (A), R29.1
- new net: D3.2 (A), R13.1
- new net: Q4.5 (B1), R23.1
- new net: Q3.2 (B), U7.3
- new net: Q3.3 (E), R20.2, U7.2 (-)
- new net: C10.1, F2.1, L2.1, U4.4 (Vin)
- new net: D4.2 (A), L2.2, U4.3 (SW), U4.6 (TAB)
- new net: Q1.3 (E), R18.2, U5.2 (-)
- new net: Q1.2 (B), U5.3
- new net: R20.2, SW2.3, SW2.4
- new net: J10.2 (D-), U9.6 (UD-)
- new net: J10.3 (D+), U9.5 (UD+)
- new net: Q4.2 (B), U8.3
- new net: D111.2 (A), R25.2
- new net: D5.2 (A), R28.1
- new net: D7.2 (A), R30.1
- new net: R14.2, R15.1, R16.1, R17.1, U4.5 (FB)
- new net: Q2.2 (B), U6.3
- new net: Q2.3 (E), R19.2, U6.2 (-)
- new net: Q6.3 (E), R23.2, U10.2 (-)
- new net: Q6.2 (B), U10.3
- new net: JP4.2 (B), R26.2
- new net: R21.2, SW3.3, SW3.4
- new net +3V3: C19.1, C20.1, R22.1, R24.1, U10.2 (VDD)
- new net 16V: J8.6 (Pin_6), R15.2
- new net 20V: J8.5 (Pin_5), R16.2
- new net 24V: J8.4 (Pin_4), R17.2
- new net 3.3V_Disp: C16.1, C17.1, R30.2, U13.5 (Vout), U9.16 (VCC), U9.4 (V3)
- new net 3.3V_Sens: C15.1, J1.3 (Pin_3), J2.3 (Pin_3), R10.2, R11.2, R29.2, U11.5 (Vout)
- new net DC: U10.23 (IO15)
- new net DTR#: Q4.4 (E1), R19.1, U9.13 (~{DTR})
- new net IO0: C17.1, Q4.3 (C1), R20.1, R22.2, U10.25 (IO0)
- new net IO2: R25.1, U10.24 (IO2)
- new net I_H1: J14.2 (Pin_2), Q5.1 (C)
- new net I_H2: J15.2 (Pin_2), Q6.1 (C)
- new net I_LED_1: J10.2 (Pin_2), Q1.1 (C)
- new net I_LED_2: J11.2 (Pin_2), Q2.1 (C)
- new net I_LED_3: J12.2 (Pin_2), Q3.1 (C)
- new net I_LED_4: J13.2 (Pin_2), Q4.1 (C), U12.12 (V_OUT_D)
- new net RES: U10.28 (IO17)
- new net RESET: C18.1, Q4.6 (C1), R21.1, R24.2, U10.3 (EN)
- new net RST#: Q4.1 (E1), R23.2, U9.14 (~{RTS})
- new net RX: U10.34 (RXD0/IO3), U9.2 (TXD)
- new net SD_cs: U10.29 (IO5)
- new net SPI_CLK: U10.30 (IO18)
- new net SPI_MISO: U10.31 (IO19)
- new net TX: U10.35 (TXD0/IO1), U9.3 (RXD)
- new net VCC_H1: C11.1, C12.1, D4.1 (K), J8.1 (Pin_1), J8.2 (Pin_2), J8.3 (Pin_3), J9.2 (Pin_2)
- new net V_H_1: U12.6 (V_OUT_E), U9.1 (+)
- new net V_H_2: U10.1 (+), U12.11 (V_OUT_F)
- new net V_LED_1: U12.4 (V_OUT_A), U5.1 (+)
- new net V_LED_2: U12.13 (V_OUT_B), U6.1 (+)
- new net V_LED_3: U12.5 (V_OUT_C), U7.1 (+)
- new net V_LED_4: U8.1 (+)
- new net V_USB: F1.2
- new net V_in: F1.1, J10.1 (VBUS)
- new net scl: U10.36 (IO22)
- new net sda: U10.33 (IO21)
- new net spi_mosi: U10.37 (IO23)
- no-connect marks 0 -> 6
Other:
- note added: "Auto reset"
- note added: "Conectores Entrada"
- note added: "Conectores Salida"
- note added: "Driver de corriente"
- note added: "ESP32-WROOM-32D"
- note added: "I2C DAC"
- note added: "If DTR is Low, toggling RTS from High to Low reset to run mode. If RTS is High, toggling DTR from Low to High reset to bootloader. Boot Mode Configuration: Pin Default Boot Download GPIO0 1 1 0 U0TXD 1 1 x GPIO2 0 x 0 GPIO4 0 x x MTDO 1 x x GPIO5 1 1 x If U0TXD, GPIO2, GPIO5 are floating, GPIO0 determines boot mode."
- note added: "Selector de voltaje"
- note added: "Switches"
- note added: "Tabla de pines ---------------- SPI_MOSI - GPIO23 SPI_MISO - GPIO19 SPI_SCK - GPIO18 CS_LORA - GPIO15 CS_SD - GPIO5 I2C_SDA - GPIO21 I2C_SCL - GPIO22 EN_VDL - EN_VS -"
- note added: "Test Points"
- note added: "USB to Serial"
- note added: "Up Voltaqe"
- note removed: "Conectores"
- moved on the sheet: C6, C7, D1, D2, F1, J1, J2, JP2, JP3, L1, R10, R11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

Commit message: ajustes_esquematico
Parts:
- removed C6: 680u, symbol Device:C
- removed C7: 330u, symbol Device:C
- removed D1: D_Schottky, symbol Device:D_Schottky
- removed D2: LED, symbol Device:LED
- removed F1: Fuse, symbol Device:Fuse
- removed J6: TP-3.3V, symbol Connector:Conn_01x02_Pin
- removed J8: Selector voltaje, symbol Connector_Generic:Conn_02x03_Counter_Clockwise
- removed L1: 68u, symbol Device:L
- removed U2: ~, Package_TO_SOT_SMD:TO-263-5_TabPin6, symbol IoWLabs:LM2596
- added 5V1: 5V, TestPoint:TestPoint_Loop_D2.50mm_Drill1.0mm_LowProfile, symbol Connector:Conn_01x01_Pin
- added C4, C8: 22u, Capacitor_SMD:C_0805_2012Metric, symbol IoWLabs:C
- added D1, D106: LED, LED_SMD:LED_0603_1608Metric, symbol Device:LED
- added D104, D105: D_Schottky, Diode_SMD:D_SMA, symbol Device:D_Schottky
- added J17: TP-3.3V, symbol Connector:Conn_01x02_Pin
- added J18: TP-3.3V-Sens, symbol Connector:Conn_01x02_Pin
- added J19: TP-3.3V-Disp, symbol Connector:Conn_01x02_Pin
- added L2: 22u, Inductor_SMD:L_Bourns_SRP7028A_7.3x6.6mm, symbol Device:L
- added Q1: Q_PMOS_GSD, Package_TO_SOT_SMD:SOT-23, symbol Device:Q_PMOS_GSD
- added R10: 7K5, Resistor_SMD:R_0603_1608Metric, symbol IoWLabs:RES
- added R11: 1K, Resistor_SMD:R_0603_1608Metric, symbol IoWLabs:RES
- added R13: 470, Resistor_SMD:R_0603_1608Metric, symbol IoWLabs:RES
- added R6: 10K, Resistor_SMD:R_0603_1608Metric, symbol IoWLabs:RES
- added SW3: SW_SP3T, symbol Switch:SW_SP3T
- added U4: MT3608, Package_TO_SOT_SMD:SOT-23-6, symbol Regulator_Switching:MT3608
- C1, C2, C3, C4, C5: footprint (none) -> Capacitor_SMD:C_0603_1608Metric
- C10, C11, C14, C15, C16, C17, C8, C9: footprint (none) -> Capacitor_SMD:C_0805_2012Metric
- C12: value C_Polarized -> 220u; footprint (none) -> Capacitor_SMD:C_0805_2012Metric
- C13: value C_Polarized -> 47u; footprint (none) -> Capacitor_SMD:C_0805_2012Metric
- D3, D5, D6, D7: footprint (none) -> LED_SMD:LED_0603_1608Metric
- F2: footprint (none) -> Fuse:Fuse_1206_3216Metric
- R1, R12, R13, R2, R3, R4, R5, R6, R7, R8, R9: footprint (none) -> Resistor_SMD:R_0603_1608Metric
- R10, R11: footprint (none) -> Resistor_SMD:R_0603_1608Metric_Pad0.98x0.95mm_HandSolder
Connections:
- net scl is gone; now on net SCL: U10.36 (IO22)
- net sda is gone; now on net SDA: U10.33 (IO21)
- net +3V3: no longer C19.1, C20.1, U10.2 (VDD)
- net 16V: now also SW3.1
- net 20V: now also SW3.2
- net 24V: now also SW3.4
- net 3.3V: now also J17.2 (Pin_2)
- net 3.3V_Disp: now also C19.1, C20.1, U10.2 (VDD), J19.2 (Pin_2)
- net 3.3V_Sens: now also J18.2 (Pin_2)
- net 5V: now also D105.1 (K), Q1.2 (S); no longer R12.2
- net GND: now also C4.2, C8.2, D1.1 (K), D106.1 (K), J17.1 (Pin_1), J18.1 (Pin_1), J19.1 (Pin_1), R11.2, R6.2, U4.2 (GND)
- net Temp1: now also C4.1, R1.1
- net Temp2: now also C3.1, R2.1
- net VCC_H1: now also SW3.3
- net V_PWR: now also C4.1, L2.1, U4.4 (EN), U4.5 (IN)
- net V_USB: now also R12.2, D105.2 (A), Q1.1 (G), R6.1
- net at R12.1: now also D1.2 (A)
- net DC: no longer names the net of U10.23 (IO15)
- net RES: no longer names the net of U10.28 (IO17)
- net V_in: no longer names the net of F1.1, J10.1 (VBUS)
- new net: D106.2 (A), R13.2
- new net 5V_IN: 5V1.1 (Pin_1), C8.1, D104.1 (K), Q1.3 (D), R10.1, R13.1
- new net FB_5V: R10.2, R11.1, U4.3 (FB)
- new net SW_5V: D104.2 (A), L2.2, U4.1 (SW)
Other:
- note added: "DC-DC 5V"
- note added: "Load sharing"
- note added: "V_out = 0.6(R39/R40 + 1)"
- note removed: "5V"
- moved on the sheet: C1, C16, C17, C18, C2, C3, C4, C5, F1, J10, J9, JP1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

Commit message: modificación
Parts:
- R18, R19, R20, R21, R22, R23: value 3.3 -> 5; footprint (none) -> Package_TO_SOT_SMD:TO-263-2
Connections:
- net 3.3V: no longer U12.8 (V_REF)
- net 5V: now also U12.8 (V_REF)
Changed lines of the file:
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@@
     )
   )
-  (global_label "3.3V" (shape input) (at 248.285 92.075 180) (fields_autoplaced)
+  (global_label "V_LED_3" (shape input) (at 29.21 173.355 180) (fields_autoplaced)
     (effects (font (size 1.27 1.27)) (justify right))
-    (property "Intersheetrefs" "${INTERSHEET_REFS}" (at 241.1874 92.075 0)
+    (property "Intersheetrefs" "${INTERSHEET_REFS}" (at 18.5444 173.355 0)
       (effects (font (size 1.27 1.27)) (justify right) hide)
     )
   )
-  (global_label "V_LED_3" (shape input) (at 29.21 173.355 180) (fields_autoplaced)
+  (global_label "5V" (shape input) (at 248.285 92.075 180) (fields_autoplaced)
     (effects (font (size 1.27 1.27)) (justify right))
-    (property "Intersheetrefs" "${INTERSHEET_REFS}" (at 18.5444 173.355 0)
+    (property "Intersheetrefs" "${INTERSHEET_REFS}" (at 243.0017 92.075 0)
       (effects (font (size 1.27 1.27)) (justify right) hide)
     )
@@
       (effects (font (size 1.27 1.27)) (justify right))
     )
-    (property "Value" "3.3" (at 119.38 191.77 0)
+    (property "Value" "5" (at 119.38 191.77 0)
       (effects (font (size 1.27 1.27)) (justify right))
     )
-    (property "Footprint" "" (at 119.253 190.5 90)
+    (property "Footprint" "Package_TO_SOT_SMD:TO-263-2" (at 119.253 190.5 90)
       (effects (font (size 1.27 1.27)) hide)
     )
@@
   (symbol (lib_id "Device:R") (at 59.69 150.495 180) (unit 1)
     (in_bom yes) (on_board yes) (dnp no) (fields_autoplaced)
-    (property "Reference" "R18" (at 61.595 149.225 0)
+    (property "Reference" "R18" (at 62.23 149.225 0)
       (effects (font (size 1.27 1.27)) (justify right))
     )
-    (property "Value" "3.3" (at 61.595 151.765 0)
+    (property "Value" "5" (at 62.23 151.765 0)
       (effects (font (size 1.27 1.27)) (justify right))
     )
-    (property "Footprint" "" (at 61.468 150.495 90)
+    (property "Footprint" "Package_TO_SOT_SMD:TO-263-2" (at 61.468 150.495 90)
       (effects (font (size 1.27 1.27)) hide)
     )
@@
   (symbol (lib_id "Device:R") (at 59.69 230.505 180) (unit 1)
     (in_bom yes) (on_board yes) (dnp no) (fields_autoplaced)
-    (property "Reference" "R22" (at 61.595 229.235 0)
+    (property "Reference" "R22" (at 62.23 229.235 0)
       (effects (font (size 1.27 1.27)) (justify right))
     )
-    (property "Value" "3.3" (at 61.595 231.775 0)
+    (property "Value" "5" (at 62.23 231.775 0)
       (effects (font (size 1.27 1.27)) (justify right))
     )
-    (property "Footprint" "" (at 61.468 230.505 90)
+    (property "Footprint" "Package_TO_SOT_SMD:TO-263-2" (at 61.468 230.505 90)
       (effects (font (size 1.27 1.27)) hide)
     )
@@
       (effects (font (size 1.27 1.27)) (justify right))
     )
-    (property "Value" "3.3" (at 62.23 191.77 0)
+    (property "Value" "5" (at 62.23 191.77 0)
       (effects (font (size 1.27 1.27)) (justify right))
     )
-    (property "Footprint" "" (at 62.103 190.5 90)
+    (property "Footprint" "Package_TO_SOT_SMD:TO-263-2" (at 62.103 190.5 90)
       (effects (font (size 1.27 1.27)) hide)
     )
@@
   (symbol (lib_id "Device:R") (at 116.84 150.495 180) (unit 1)
     (in_bom yes) (on_board yes) (dnp no) (fields_autoplaced)
-    (property "Reference" "R19" (at 118.745 149.225 0)
+    (property "Reference" "R19" (at 119.38 149.225 0)
       (effects (font (size 1.27 1.27)) (justify right))
     )
-    (property "Value" "3.3" (at 118.745 151.765 0)
+    (property "Value" "5" (at 119.38 151.765 0)
       (effects (font (size 1.27 1.27)) (justify right))
     )
-    (property "Footprint" "" (at 118.618 150.495 90)
+    (property "Footprint" "Package_TO_SOT_SMD:TO-263-2" (at 118.618 150.495 90)
       (effects (font (size 1.27 1.27)) hide)
     )
@@
   (symbol (lib_id "Device:R") (at 116.84 230.505 180) (unit 1)
     (in_bom yes) (on_board yes) (dnp no) (fields_autoplaced)
-    (property "Reference" "R23" (at 118.745 229.235 0)
+    (property "Reference" "R23" (at 119.38 229.235 0)
       (effects (font (size 1.27 1.27)) (justify right))
     )
-    (property "Value" "3.3" (at 118.745 231.775 0)
+    (property "Value" "5" (at 119.38 231.775 0)
       (effects (font (size 1.27 1.27)) (justify right))
     )
-    (property "Footprint" "" (at 118.618 230.505 90)
+    (property "Footprint" "Package_TO_SOT_SMD:TO-263-2" (at 118.618 230.505 90)
       (effects (font (size 1.27 1.27)) hide)
     )

Commit message: placa
Parts:
- removed 5V1: 5V, TestPoint:TestPoint_Loop_D2.50mm_Drill1.0mm_LowProfile, symbol Connector:Conn_01x01_Pin
- removed J10: LED_1, symbol Connector:Conn_01x02_Pin
- removed J11: LED_2, symbol Connector:Conn_01x02_Pin
- removed J12: LED_3, symbol Connector:Conn_01x02_Pin
- removed J13: LED_4, symbol Connector:Conn_01x02_Pin
- removed J14: H1, symbol Connector:Conn_01x02_Pin
- removed J15: H2, symbol Connector:Conn_01x02_Pin
- removed SW3: SW_SP3T, symbol Switch:SW_SP3T
- removed U10, U5, U6, U7, U8, U9: ${SIM.PARAMS}, symbol Simulation_SPICE:OPAMP
- added J10: H1, Connector_JST:JST_XH_B3B-XH-A_1x03_P2.50mm_Vertical, symbol Connector:Conn_01x03_Pin
- added J11: H2, Connector_JST:JST_XH_B3B-XH-A_1x03_P2.50mm_Vertical, symbol Connector:Conn_01x03_Pin
- added J12: LED_4, Connector_JST:JST_XH_B3B-XH-A_1x03_P2.50mm_Vertical, symbol Connector:Conn_01x03_Pin
- added J13: LED_2, Connector_JST:JST_XH_B3B-XH-A_1x03_P2.50mm_Vertical, symbol Connector:Conn_01x03_Pin
- added J6: LED_1, Connector_JST:JST_XH_B3B-XH-A_1x03_P2.50mm_Vertical, symbol Connector:Conn_01x03_Pin
- added J8: LED_3, Connector_JST:JST_XH_B3B-XH-A_1x03_P2.50mm_Vertical, symbol Connector:Conn_01x03_Pin
- added U2, U5, U6: TLC272, Package_SO:SOIC-8_3.9x4.9mm_P1.27mm, symbol Amplifier_Operational:TLC272
- added U7: ~, IoWLabsConnectors:Switch SP3T SS13D07L2B, symbol IoWLabsConnectors:SS13D07L2B
- C12: footprint Capacitor_SMD:C_0805_2012Metric -> Capacitor_SMD:CP_Elec_10x10.5
- C13: footprint Capacitor_SMD:C_0805_2012Metric -> Capacitor_SMD:CP_Elec_6.3x7.7
- D4: footprint (none) -> Diode_SMD:D_SMA
- J1, J2, J3: footprint (none) -> Connector_JST:JST_XH_B3B-XH-A_1x03_P2.50mm_Vertical
- J17, J18, J19, J4, J5, J7, J9: footprint (none) -> Connector_JST:JST_XH_B2B-XH-A_1x02_P2.50mm_Vertical
- JP1, JP2, JP3, JP4: footprint (none) -> Jumper:SolderJumper-2_P1.3mm_Open_RoundedPad1.0x1.5mm
- L2: footprint (none) -> Inductor_SMD:L_12x12mm_H8mm
- Q1, Q2, Q3, Q4, Q5, Q6: footprint (none) -> Package_TO_SOT_SMD:SOT-223-3_TabPin2
- R10, R11: footprint Resistor_SMD:R_0603_1608Metric_Pad0.98x0.95mm_HandSolder -> Resistor_SMD:R_0603_1608Metric
- R14, R15, R16, R17, R24, R25, R26, R27, R28, R29, R30: footprint (none) -> Resistor_SMD:R_0603_1608Metric
- R18, R19, R20, R21, R22, R23: footprint Package_TO_SOT_SMD:TO-263-2 -> IoWLabs:TO-263-3 TAB 3
Connections:
- net 16V: now also U7.1
- net 20V: now also U7.3
- net 24V: now also U7.4
- net GND: now also J10.1 (Pin_1), J11.1 (Pin_1), J12.1 (Pin_1), J13.1 (Pin_1), J6.1 (Pin_1), J8.1 (Pin_1), U2.4 (V-), U5.4 (V-), U6.4 (V-)
- net I_H1: now also J10.2 (Pin_2)
- net I_H2: now also J11.2 (Pin_2)
- net I_LED_1: now also J6.2 (Pin_2)
- net I_LED_2: now also J13.2 (Pin_2)
- net I_LED_3: now also J8.2 (Pin_2)
- net I_LED_4: now also J12.2 (Pin_2); no longer U12.12 (V_OUT_D)
- net VCC_H1: now also J10.3 (Pin_3), J11.3 (Pin_3), J12.3 (Pin_3), J13.3 (Pin_3), J6.3 (Pin_3), J8.3 (Pin_3), U7.2
- net V_H_1: now also U12.13 (V_OUT_B), U6.3 (+); no longer U12.6 (V_OUT_E)
- net V_H_2: now also U6.5 (+)
- net V_LED_1: now also U2.3 (+)
- net V_LED_2: now also U12.5 (V_OUT_C), U2.5 (+); no longer U12.13 (V_OUT_B)
- net V_LED_3: now also U12.6 (V_OUT_E), U5.3 (+); no longer U12.5 (V_OUT_C)
- net V_LED_4: now also U12.12 (V_OUT_D), U5.5 (+)
- net V_PWR: now also U2.8 (V+), U5.8 (V+), U6.8 (V+)
- net at Q5.3 (E), R22.2: now also U6.2 (-)
- net at Q5.2 (B): now also U6.1
- net at Q4.3 (E), R21.2: now also U5.6 (-)
- net at Q3.2 (B): now also U5.1
- net at Q3.3 (E), R20.2: now also U5.2 (-)
- net at Q1.3 (E), R18.2: now also U2.2 (-)
- net at Q1.2 (B): now also U2.1
- net at Q4.2 (B): now also U5.7
- net at Q2.2 (B): now also U2.7
- net at Q2.3 (E), R19.2: now also U2.6 (-)
- net at Q6.3 (E), R23.2: now also U6.6 (-)
- net at Q6.2 (B): now also U6.7

Commit message: pcb
Parts:
- added H1, H2, H3, H4: MountingHole, MountingHole:MountingHole_3.2mm_M3, symbol Mechanical:MountingHole
Changed lines of the file:
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@@
     )
   )
+  (symbol (lib_id "Mechanical:MountingHole") (at 453.39 37.465 0) (unit 1)
+    (in_bom yes) (on_board yes) (dnp no) (fields_autoplaced)
+    (property "Reference" "H3" (at 455.93 36.195 0)
+      (effects (font (size 1.27 1.27)) (justify left))
+    )
+    (property "Value" "MountingHole" (at 455.93 38.735 0)
+      (effects (font (size 1.27 1.27)) (justify left))
+    )
+    (property "Footprint" "MountingHole:MountingHole_3.2mm_M3" (at 453.39 37.465 0)
+      (effects (font (size 1.27 1.27)) hide)
+    )
+    (property "Datasheet" "~" (at 453.39 37.465 0)
+      (effects (font (size 1.27 1.27)) hide)
+    )
+    (instances
+      (project "FluOpti_V3.0"
+        (path "/a7d210b0-29ee-4db1-96c4-600f3ef4cf17"
+          (reference "H3") (unit 1)
+        )
+      )
+    )
+  )
   (symbol (lib_id "power:GND") (at 315.595 84.455 0) (unit 1)
     (in_bom yes) (on_board yes) (dnp no) (fields_autoplaced)
@@
     )
   )
+  (symbol (lib_id "Mechanical:MountingHole") (at 453.39 44.45 0) (unit 1)
+    (in_bom yes) (on_board yes) (dnp no) (fields_autoplaced)
+    (property "Reference" "H4" (at 455.93 43.18 0)
+      (effects (font (size 1.27 1.27)) (justify left))
+    )
+    (property "Value" "MountingHole" (at 455.93 45.72 0)
+      (effects (font (size 1.27 1.27)) (justify left))
+    )
+    (property "Footprint" "MountingHole:MountingHole_3.2mm_M3" (at 453.39 44.45 0)
+      (effects (font (size 1.27 1.27)) hide)
+    )
+    (property "Datasheet" "~" (at 453.39 44.45 0)
+      (effects (font (size 1.27 1.27)) hide)
+    )
+    (instances
+      (project "FluOpti_V3.0"
+        (path "/a7d210b0-29ee-4db1-96c4-600f3ef4cf17"
+          (reference "H4") (unit 1)
+        )
+      )
+    )
+  )
   (symbol (lib_id "Device:R") (at 89.535 68.58 270) (unit 1)
     (in_bom yes) (on_board yes) (dnp no) (fields_autoplaced)
@@
     )
   )
+  (symbol (lib_id "Mechanical:MountingHole") (at 453.39 25.4 0) (unit 1)
+    (in_bom yes) (on_board yes) (dnp no) (fields_autoplaced)
+    (property "Reference" "H1" (at 455.93 24.13 0)
+      (effects (font (size 1.27 1.27)) (justify left))
+    )
+    (property "Value" "MountingHole" (at 455.93 26.67 0)
+      (effects (font (size 1.27 1.27)) (justify left))
+    )
+    (property "Footprint" "MountingHole:MountingHole_3.2mm_M3" (at 453.39 25.4 0)
+      (effects (font (size 1.27 1.27)) hide)
+    )
+    (property "Datasheet" "~" (at 453.39 25.4 0)
+      (effects (font (size 1.27 1.27)) hide)
+    )
+    (instances
+      (project "FluOpti_V3.0"
+        (path "/a7d210b0-29ee-4db1-96c4-600f3ef4cf17"
+          (reference "H1") (unit 1)
+        )
+      )
+    )
+  )
   (symbol (lib_id "Device:C") (at 297.18 77.47 0) (unit 1)
     (in_bom yes) (on_board yes) (dnp no) (fields_autoplaced)
@@
         )
       )
+    )
+  )
+  (symbol (lib_id "Mechanical:MountingHole") (at 453.39 31.75 0) (unit 1)
+    (in_bom yes) (on_board yes) (dnp no) (fields_autoplaced)
+    (property "Reference" "H2" (at 455.93 30.48 0)
+      (effects (font (size 1.27 1.27)) (justify left))
+    )
+    (property "Value" "MountingHole" (at 455.93 33.02 0)
+      (effects (font (size 1.27 1.27)) (justify left))
+    )
+    (property "Footprint" "MountingHole:MountingHole_3.2mm_M3" (at 453.39 31.75 0)
+      (effects (font (size 1.27 1.27)) hide)
+    )
+    (property "Datasheet" "~" (at 453.39 31.75 0)
+      (effects (font (size 1.27 1.27)) hide)
+    )
+    (instances
+      (project "FluOpti_V3.0"
+        (path "/a7d210b0-29ee-4db1-96c4-600f3ef4cf17"
+          (reference "H2") (unit 1)
+        )
+      )
