File: hardware/FluOpti_V3.0/FluOpti_V3.0.kicad_sch (KiCad schematic)
At the start: 125 parts, among them J1 Sensor1, J10 H1, J10 USB_B_Micro, J11 H2, J12 LED_4, J13 LED_2, J17 TP-3.3V, J18 TP-3.3V-Sens, J19 TP-3.3V-Disp, J2 Sensor2, J3 I2C_IN, J4 PWR_IN, J5 TP-5V, J6 LED_1, J7 TP-PWR_IN, J8 LED_3, J9 TP-VCC_H1, Q1 NPN, Q1 Q_PMOS_GSD, Q2 NPN, Q3 NPN, Q4 NPN, Q4 Q_Dual_NPN_NPN_BRT_E1B1C2E2B2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, Q5 NPN, Q6 NPN, SW2 SW_DIP_x02, SW3 SW_DIP_x02, U1 ADS1115IDGS, U10 ESP32-WROOM-32D, U11 AP2112K-3.3TRG1, U12 AD5659R, U13 AP2112K-3.3TRG1, U2 TLC272, U3 AP2112K-3.3TRG1, U4 MT3608, U4 XL6008, U5 TLC272, U6 TLC272, U9 CH340C

Commit message: adding some documentation
Parts:
- removed C14, C15, C16, C17: 1u, Capacitor_SMD:C_0805_2012Metric, symbol Device:C
- removed D6, D7: LED, LED_SMD:LED_0603_1608Metric, symbol Device:LED
- removed J10: H1, Connector_JST:JST_XH_B3B-XH-A_1x03_P2.50mm_Vertical, symbol Connector:Conn_01x03_Pin
- removed J11: H2, Connector_JST:JST_XH_B3B-XH-A_1x03_P2.50mm_Vertical, symbol Connector:Conn_01x03_Pin
- removed R29, R30: 10, Resistor_SMD:R_0603_1608Metric, symbol Device:R
- removed U11, U13: AP2112K-3.3TRG1, IoWLabs:SOT-25, symbol IoWLabs:AP2112K-3.3TRG1-SOT25
- added J14, J15, J20, J21, J22, J23: HDR-2x1, symbol IoWLabsConnectors:HDR-2x1
- J4: footprint Connector_JST:JST_XH_B2B-XH-A_1x02_P2.50mm_Vertical -> IoWLabsConnectors:Tb-2x1-5p-TH-V
Connections:
- net 3.3V: now also C19.1, C20.1, U10.2 (VDD), U9.16 (VCC), U9.4 (V3)
- net 3.3V_Disp: no longer C19.1, C20.1, U10.2 (VDD), U9.16 (VCC), U9.4 (V3)
- net GND: no longer J12.1 (Pin_1), J13.1 (Pin_1), J6.1 (Pin_1), J8.1 (Pin_1)
- net I_H1: now also J22.2
- net I_H2: now also J23.2
- net I_LED_1: now also J14.2, J21.2; no longer J6.2 (Pin_2)
- net I_LED_2: now also J15.2; no longer J13.2 (Pin_2)
- net I_LED_3: no longer J8.2 (Pin_2)
- net I_LED_4: now also J20.2; no longer J12.2 (Pin_2)
- net VCC_H1: now also J22.1, J23.1
- net V_PWR: now also J12.1 (Pin_1), J13.1 (Pin_1), J6.1 (Pin_1), J8.1 (Pin_1)
- new net VCC_LED_1: J14.1, J6.2 (Pin_2)
- new net VCC_LED_2: J13.2 (Pin_2), J15.1
- new net VCC_LED_3: J20.1, J8.2 (Pin_2)
- new net VCC_LED_4: J12.2 (Pin_2), J21.1
Other:
- moved on the sheet: J12, J13, J6, J8
